Commit message: xacro modell, lidar javítva, RVIZ térkép tökéletes

File: urdf/mecanum.xacro (robot description, xacro)
@@ -163,5 +163,5 @@
     <parent link="base_link" />
     <child link="base_scan" />
-    <origin xyz="0 0 0.1" rpy="0 0 3.1415" />
+    <origin xyz="0.175 0 0.1" rpy="0 0 0" />
 </joint>
 <gazebo reference="base_scan">

Commit message: javított xacro a modell méretei alapján, lidar 270 fokos

File: urdf/mecanum.xacro (robot description, xacro)
@@ -3,8 +3,8 @@
 <!-- <xacro:include filename="hokuyo_ust10.xacro" /> -->
 <xacro:property name="radius" value="0.05" />
-<xacro:property name="length" value="0.08" />
-<xacro:property name="box_length" value="0.5" />
-<xacro:property name="box_width" value="0.3" />
-<xacro:property name="box_height" value="0.1" />
+<xacro:property name="length" value="0.06" />
+<xacro:property name="box_length" value="0.3" />
+<xacro:property name="box_width" value="0.2" />
+<xacro:property name="box_height" value="0.09" />
 <material name="blue">
  <color rgba="0 0 0.8 1" />
@@ -21,7 +21,7 @@
 <link name="front_right_wheel">
     <visual>
-        <origin xyz="0 0 0.05" rpy="1.57075 0 0"  />
-        <geometry>
-            <mesh filename="file://$(find mecanum_launch)/meshes/Mecanum_jo.stl" scale="0.0015 0.0015 0.0015" />
+        <origin xyz="0 0 0.02" rpy="1.57075 0 0"  />
+        <geometry>
+            <mesh filename="file://$(find mecanum_launch)/meshes/Mecanum_jo.stl" scale="0.0010 0.0010 0.0010" />
         </geometry>
         <material name="black" />
@@ -40,16 +40,17 @@
     <parent link="base_link" />
     <child link="front_right_wheel" />
-    <origin xyz="0.2 -${box_width/2+length/2} -0.05" />
+    <origin xyz="0.1 -${box_width/2+length/2} -0.03" />
     <axis xyz="0 1 0" />
 </joint>
 <link name="front_left_wheel">
     <visual>
-        <origin xyz="0 0 0.05" rpy="1.57075 0 0"  />
-        <geometry>
-            <mesh filename="file://$(find mecanum_launch)/meshes/Mecanum_jo.stl" scale="0.0015 0.0015 0.0015" />
-        </geometry>
-        <material name="black" />
-    </visual>
-    <collision>
+        <origin xyz="0 0 0.02" rpy="1.57075 0 0"  />
+        <geometry>
+            <mesh filename="file://$(find mecanum_launch)/meshes/Mecanum_jo.stl" scale="0.0010 0.0010 0.0010" />
+        </geometry>
+        <material name="black" />
+    </visual>
+    <collision>
+        <origin xyz="0 0 0" rpy="1.57075 0 0"  />
         <geometry>
             <cylinder length="${length}" radius="${radius}" />
@@ -64,16 +65,17 @@
     <parent link="base_link" />
     <child link="front_left_wheel" />
-    <origin xyz="0.2 ${box_width/2+length/2} -0.05" />
+    <origin xyz="0.1 ${box_width/2+length/2} -0.03" />
     <axis xyz="0 1 0" />
 </joint>
 <link name="rear_left_wheel">
     <visual>
-        <origin xyz="0 0 0.05" rpy="1.57075 0 0"  />
-        <geometry>
-            <mesh filename="file://$(find mecanum_launch)/meshes/Mecanum_jo.stl" scale="0.0015 0.0015 0.0015" />
-        </geometry>
-        <material name="black" />
-    </visual>
-    <collision>
+        <origin xyz="0 0 0.02" rpy="1.57075 0 0"  />
+        <geometry>
+            <mesh filename="file://$(find mecanum_launch)/meshes/Mecanum_jo.stl" scale="0.0010 0.0010 0.0010" />
+        </geometry>
+        <material name="black" />
+    </visual>
+    <collision>
+        <origin xyz="0 0 0" rpy="1.57075 0 0"  />
         <geometry>
             <cylinder length="${length}" radius="${radius}" />
@@ -88,16 +90,17 @@
     <parent link="base_link" />
     <child link="rear_left_wheel" />
-    <origin xyz="-0.2 ${box_width/2+length/2} -0.05" />
+    <origin xyz="-0.1 ${box_width/2+length/2} -0.03" />
     <axis xyz="0 1 0" />
 </joint>
 <link name="rear_right_wheel">
     <visual>
-        <origin xyz="0 0 0.05" rpy="1.57075 0 0"  />
-        <geometry>
-            <mesh filename="file://$(find mecanum_launch)/meshes/Mecanum_jo.stl" scale="0.0015 0.0015 0.0015" />
-        </geometry>
-        <material name="black" />
-    </visual>
-    <collision>
+        <origin xyz="0 0 0.02" rpy="1.57075 0 0"  />
+        <geometry>
+            <mesh filename="file://$(find mecanum_launch)/meshes/Mecanum_jo.stl" scale="0.0010 0.0010 0.0010" />
+        </geometry>
+        <material name="black" />
+    </visual>
+    <collision>
+        <origin xyz="0 0 0" rpy="1.57075 0 0"  />
         <geometry>
             <cylinder length="${length}" radius="${radius}" />
@@ -112,9 +115,10 @@
     <parent link="base_link" />
     <child link="rear_right_wheel" />
-    <origin xyz="-0.2 -${box_width/2+length/2} -0.05" />
+    <origin xyz="-0.1 -${box_width/2+length/2} -0.03" />
     <axis xyz="0 1 0" />
 </joint>
 <link name="base_link">
     <visual>
+    <origin xyz="0 0 0" rpy="0 0 0"  />
         <geometry>
             <box size="${box_length} ${box_width} ${box_height}" />
@@ -123,5 +127,5 @@
     </visual>
     <collision>
-        <origin xyz="-0.02 0 0.035" rpy="0 0 0"  />
+        <origin xyz="0 0 0" rpy="0 0 0"  />
         <geometry>
             <box size="${box_length} ${box_width} ${box_height}" />
@@ -130,5 +134,5 @@
     <inertial>
         <origin xyz="-0.02 0 0.035" rpy="0 0 0" />
-        <mass value="1.0" />
+        <mass value="3.0" />
         <inertia ixx="0.00129283" ixy="0" ixz="0" iyy="0.00440742" iyz="0" izz="0.00495208" />
     </inertial>
@@ -163,5 +167,5 @@
     <parent link="base_link" />
     <child link="base_scan" />
-    <origin xyz="0.175 0 0.1" rpy="0 0 0" />
+    <origin xyz="0.1 0 0.09" rpy="0 0 0" />
 </joint>
 <gazebo reference="base_scan">
@@ -176,6 +180,6 @@
                     <samples>500</samples>
                     <resolution>0.72</resolution>
-                    <min_angle>0.0</min_angle>
-                    <max_angle>6.28319</max_angle>
+                    <min_angle>-2.3562</min_angle>
+                    <max_angle>2.3562</max_angle>
                 </horizontal>
             </scan>
@@ -183,5 +187,5 @@
                 <min>0.120</min>
                 <max>10</max>
-                <resolution>0.015</resolution>
+                <resolution>0.25</resolution>
             </range>
             <noise>

Commit message: Dipterv_B_nem tudom hol tartottam

File: urdf/mecanum.xacro (robot description, xacro)
@@ -3,5 +3,5 @@
 <!-- <xacro:include filename="hokuyo_ust10.xacro" /> -->
 <xacro:property name="radius" value="0.05" />
-<xacro:property name="length" value="0.06" />
+<xacro:property name="length" value="0.05" />
 <xacro:property name="box_length" value="0.3" />
 <xacro:property name="box_width" value="0.2" />
@@ -150,5 +150,5 @@
             <mesh filename="file://$(find mecanum_launch)/meshes/sensors/hokuyo_ust10.stl" scale="1 1 1" />
         </geometry>
-        <material name="white" />
+        <material name="black" />
     </visual>
     <collision>

Commit message: RVIZ-ben moveit interactive marker és plan+execute működik, csak ha a fixed frame base_link-re át van állítva

File: urdf/mecanum.xacro (robot description, xacro)
@@ -1,10 +1,12 @@
 <?xml version="1.0"?>
-<robot xmlns:xacro="https://www.ros.org/wiki/xacro" name="mecanum">
+<robot xmlns:xacro="https://www.ros.org/wiki/xacro" name="mecanum" xmlns:ignition="http://gazebosim.org/schema">
 <!-- <xacro:include filename="hokuyo_ust10.xacro" /> -->
 <xacro:property name="radius" value="0.05" />
 <xacro:property name="length" value="0.05" />
+<xacro:property name="mass" value="0.4" />
 <xacro:property name="box_length" value="0.3" />
 <xacro:property name="box_width" value="0.2" />
 <xacro:property name="box_height" value="0.09" />
+<xacro:property name="box_mass" value="3.0" />
 <material name="blue">
  <color rgba="0 0 0.8 1" />
@@ -19,13 +21,17 @@
  <color rgba="1 1 1 1" />
 </material>
+<material name="orange">
+ <color rgba="1 0.5 0 1" />
+</material>
 <link name="front_right_wheel">
     <visual>
-        <origin xyz="0 0 0.02" rpy="1.57075 0 0"  />
-        <geometry>
-            <mesh filename="file://$(find mecanum_launch)/meshes/Mecanum_jo.stl" scale="0.0010 0.0010 0.0010" />
-        </geometry>
-        <material name="black" />
-    </visual>
-    <collision>
+        <origin xyz="0 0 0" rpy="1.57075 0 0"  />
+        <geometry>
+            <mesh filename="file://$(find mecanum_moveit_launch)/meshes/Mecanum_jo.stl" scale="0.0010 0.0010 0.0010" />
+        </geometry>
+        <material name="black" />
+    </visual>
+    <collision>
+        <origin xyz="0 0 0" rpy="1.57075 0 0"  />
         <geometry>
             <cylinder length="${length}" radius="${radius}" />
@@ -33,6 +39,6 @@
     </collision>
     <inertial>
-        <mass value="0.3"/>
-        <inertia ixx="1e-3" ixy="0" ixz="0" iyy="1e-3" iyz="0" izz="1e-3" />
+        <mass value="${mass}"/>
+        <inertia ixx="${1/12*mass*(3*radius*radius+length*length)}" ixy="0" ixz="0" iyy="${1/2*mass*radius*radius}" iyz="0" izz="${1/12*mass*(3*radius*radius+length*length)}" />
     </inertial>
 </link>
@@ -45,7 +51,7 @@
 <link name="front_left_wheel">
     <visual>
-        <origin xyz="0 0 0.02" rpy="1.57075 0 0"  />
-        <geometry>
-            <mesh filename="file://$(find mecanum_launch)/meshes/Mecanum_jo.stl" scale="0.0010 0.0010 0.0010" />
+        <origin xyz="0 0 0" rpy="1.57075 0 0"  />
+        <geometry>
+            <mesh filename="file://$(find mecanum_moveit_launch)/meshes/Mecanum_jo.stl" scale="0.0010 0.0010 0.0010" />
         </geometry>
         <material name="black" />
@@ -58,6 +64,6 @@
     </collision>
     <inertial>
-        <mass value="0.3"/>
-        <inertia ixx="1e-3" ixy="0" ixz="0" iyy="1e-3" iyz="0" izz="1e-3" />
+        <mass value="${mass}"/>
+        <inertia ixx="${1/12*mass*(3*radius*radius+length*length)}" ixy="0" ixz="0" iyy="${1/2*mass*radius*radius}" iyz="0" izz="${1/12*mass*(3*radius*radius+length*length)}" />
     </inertial>
 </link>
@@ -70,7 +76,7 @@
 <link name="rear_left_wheel">
     <visual>
-        <origin xyz="0 0 0.02" rpy="1.57075 0 0"  />
-        <geometry>
-            <mesh filename="file://$(find mecanum_launch)/meshes/Mecanum_jo.stl" scale="0.0010 0.0010 0.0010" />
+        <origin xyz="0 0 0" rpy="1.57075 0 0"  />
+        <geometry>
+            <mesh filename="file://$(find mecanum_moveit_launch)/meshes/Mecanum_jo.stl" scale="0.0010 0.0010 0.0010" />
         </geometry>
         <material name="black" />
@@ -83,6 +89,6 @@
     </collision>
     <inertial>
-        <mass value="0.3"/>
-        <inertia ixx="1e-3" ixy="0" ixz="0" iyy="1e-3" iyz="0" izz="1e-3" />
+        <mass value="${mass}"/>
+        <inertia ixx="${1/12*mass*(3*radius*radius+length*length)}" ixy="0" ixz="0" iyy="${1/2*mass*radius*radius}" iyz="0" izz="${1/12*mass*(3*radius*radius+length*length)}" />
     </inertial>
 </link>
@@ -95,7 +101,7 @@
 <link name="rear_right_wheel">
     <visual>
-        <origin xyz="0 0 0.02" rpy="1.57075 0 0"  />
-        <geometry>
-            <mesh filename="file://$(find mecanum_launch)/meshes/Mecanum_jo.stl" scale="0.0010 0.0010 0.0010" />
+        <origin xyz="0 0 0" rpy="1.57075 0 0"  />
+        <geometry>
+            <mesh filename="file://$(find mecanum_moveit_launch)/meshes/Mecanum_jo.stl" scale="0.0010 0.0010 0.0010" />
         </geometry>
         <material name="black" />
@@ -108,6 +114,6 @@
     </collision>
     <inertial>
-        <mass value="0.3"/>
-        <inertia ixx="1e-3" ixy="0" ixz="0" iyy="1e-3" iyz="0" izz="1e-3" />
+        <mass value="${mass}"/>
+        <inertia ixx="${1/12*mass*(3*radius*radius+length*length)}" ixy="0" ixz="0" iyy="${1/2*mass*radius*radius}" iyz="0" izz="${1/12*mass*(3*radius*radius+length*length)}" />
     </inertial>
 </link>
@@ -134,6 +140,6 @@
     <inertial>
         <origin xyz="-0.02 0 0.035" rpy="0 0 0" />
-        <mass value="3.0" />
-        <inertia ixx="0.00129283" ixy="0" ixz="0" iyy="0.00440742" iyz="0" izz="0.00495208" />
+        <mass value="${box_mass}" />
+        <inertia ixx="${1/12*box_mass*(box_height*box_height+box_width*box_width)}" ixy="0" ixz="0" iyy="${1/12*box_mass*(box_length*box_length+box_height*box_height)}" iyz="0" izz="${1/12*box_mass*(box_length*box_length+box_width*box_width)}" />
     </inertial>
 </link>
@@ -148,5 +154,5 @@
         <origin xyz="0 0 -0.05" rpy="0 0 0"  />
         <geometry>
-            <mesh filename="file://$(find mecanum_launch)/meshes/sensors/hokuyo_ust10.stl" scale="1 1 1" />
+            <mesh filename="file://$(find mecanum_moveit_launch)/meshes/sensors/hokuyo_ust10.stl" scale="0.8 0.8 0.8" />
         </geometry>
         <material name="black" />
@@ -169,40 +175,357 @@
     <origin xyz="0.1 0 0.09" rpy="0 0 0" />
 </joint>
+<link name="link_0">
+    <visual>
+        <origin xyz="-0.005 0.010 -0.035" rpy="1.57075 0 0"  />
+        <geometry>
+            <mesh filename="file://$(find mecanum_moveit_launch)/meshes/simplify_link_0.stl" scale="0.0003 0.0003 0.0003" />
+        </geometry>
+        <material name="black" />
+    </visual>
+    <collision>
+        <origin xyz="0 0 -0.01" rpy="0 0 0"  />
+        <geometry>
+            <box size="0.1 0.1 0.04" />
+        </geometry>
+    </collision>
+    <inertial>
+        <mass value="${mass}"/>
+        <inertia ixx="${1/12*mass*(3*radius*radius+length*length)}" ixy="0" ixz="0" iyy="${1/2*mass*radius*radius}" iyz="0" izz="${1/12*mass*(3*radius*radius+length*length)}" />
+    </inertial>
+</link>
+<joint name="teto" type="fixed">
+    <parent link="base_link" />
+    <child link="link_0" />
+    <origin xyz="-0.02 0.0075 0.080" />
+    <axis xyz="0 1 0" />
+</joint>
+<link name="link_1">
+    <visual>
+        <origin xyz="-0.020 -0.030 -0.065" rpy="1.57075 0 0"  />
+        <geometry>
+            <mesh filename="file://$(find mecanum_moveit_launch)/meshes/simplify_link_1.stl" scale="-0.0003 0.0003 0.0003" />
+        </geometry>
+        <material name="orange" />
+    </visual>
+    <collision>
+        <origin xyz="0 0 -0.02" rpy="0 0 0"  />
+        <geometry>
+            <box size="0.08 0.08 0.03" />
+        </geometry>
+    </collision>
+    <inertial>
+        <mass value="${mass}"/>
+        <inertia ixx="${1/12*mass*(3*radius*radius+length*length)}" ixy="0" ixz="0" iyy="${1/2*mass*radius*radius}" iyz="0" izz="${1/12*mass*(3*radius*radius+length*length)}" />
+    </inertial>
+</link>
+<joint name="rob_joint_1" type="revolute">
+    <parent link="link_0" />
+    <child link="link_1" />
+    <origin xyz="0 0 0.060" rpy="0 0 0"/>
+    <axis xyz="0 0 1" />
+    <limit lower="-2.967" upper="2.967" effort="10" velocity="1.0"/>
+</joint>
+<link name="link_2">
+    <visual>
+        <origin xyz="0.005 -0.115 0.048" rpy="0 0 0"  />
+        <geometry>
+            <mesh filename="file://$(find mecanum_moveit_launch)/meshes/simplify_link_2.stl" scale="-0.0003 0.0003 0.0003" />
+        </geometry>
+        <material name="orange" />
+    </visual>
+    <collision>
+        <origin xyz="0 -0.05 0" rpy="1.57075 0 0"  />
+        <geometry>
+            <cylinder length="0.08" radius="0.02" />
+        </geometry>
+    </collision>
+    <inertial>
+        <mass value="${mass}"/>
+        <inertia ixx="${1/12*mass*(3*radius*radius+length*length)}" ixy="0" ixz="0" iyy="${1/2*mass*radius*radius}" iyz="0" izz="${1/12*mass*(3*radius*radius+length*length)}" />
+    </inertial>
+</link>
+<joint name="rob_joint_2" type="revolute">
+    <parent link="link_1" />
+    <child link="link_2" />
+    <origin xyz="0.01 0 0" rpy="-1.57075 0 0"/>
+    <axis xyz="0 0 1" />
+    <limit lower="-3.3161" upper="0.7854" effort="10" velocity="1.0"/>
+</joint>
+<link name="link_3">
+    <visual>
+        <origin xyz="0.015 -0.025 0.0235" rpy="0 0 0"  />
+        <geometry>
+            <mesh filename="file://$(find mecanum_moveit_launch)/meshes/simplify_link_3.stl" scale="-0.0003 0.0003 0.0003" />
+        </geometry>
+        <material name="orange" />
+    </visual>
+    <collision>
+        <origin xyz="0 0.03 0" rpy="0 1.57075 0"  />
+        <geometry>
+            <cylinder length="0.08" radius="0.02" />
+        </geometry>
+    </collision>
+    <inertial>
+        <mass value="${mass}"/>
+        <inertia ixx="${1/12*mass*(3*radius*radius+length*length)}" ixy="0" ixz="0" iyy="${1/2*mass*radius*radius}" iyz="0" izz="${1/12*mass*(3*radius*radius+length*length)}" />
+    </inertial>
+</link>
+<joint name="rob_joint_3" type="revolute">
+    <parent link="link_2" />
+    <child link="link_3" />
+    <origin xyz="0 -0.090 0" rpy="3.14 0 0" />
+    <axis xyz="0 0 1" />
+    <limit lower="-2.0944" upper="2.7227" effort="10" velocity="1.0"/>
+</joint>
+<link name="link_4">
+    <visual>
+        <origin xyz="0.04 -0.020 0.015" rpy="0 0 0"  />
+        <geometry>
+            <mesh filename="file://$(find mecanum_moveit_launch)/meshes/simplify_link_4.stl" scale="-0.0003 0.0003 0.0003" />
+        </geometry>
+        <material name="orange" />
+    </visual>
+    <collision>
+        <origin xyz="0 0 0" rpy="0 1.57075 0"  />
+        <geometry>
+            <cylinder length="0.04" radius="0.016" />
+        </geometry>
+    </collision>
+    <inertial>
+        <mass value="${mass}"/>
+        <inertia ixx="${1/12*mass*(3*radius*radius+length*length)}" ixy="0" ixz="0" iyy="${1/2*mass*radius*radius}" iyz="0" izz="${1/12*mass*(3*radius*radius+length*length)}" />
+    </inertial>
+</link>
+<joint name="rob_joint_4" type="revolute">
+    <parent link="link_3" />
+    <child link="link_4" />
+    <origin xyz="0.065 0.025 0" />
+    <axis xyz="1 0 0" />
+    <limit lower="-3.2289" upper="3.2289" effort="10" velocity="1.0"/>
+</joint>
+<link name="link_5">
+    <visual>
+        <origin xyz="0.020 -0.02 0.02" rpy="0 0 0"  />
+        <geometry>
+            <mesh filename="file://$(find mecanum_moveit_launch)/meshes/simplify_link_5.stl" scale="-0.0003 0.0003 0.0003" />
+        </geometry>
+        <material name="orange" />
+    </visual>
+    <collision>
+        <origin xyz="0.015 0 0" rpy="0 1.57075 0"  />
+        <geometry>
+            <cylinder length="0.04" radius="0.016" />
+        </geometry>
+    </collision>
+    <inertial>
+        <mass value="${mass}"/>
+        <inertia ixx="${1/12*mass*(3*radius*radius+length*length)}" ixy="0" ixz="0" iyy="${1/2*mass*radius*radius}" iyz="0" izz="${1/12*mass*(3*radius*radius+length*length)}" />
+    </inertial>
+</link>
+<joint name="rob_joint_5" type="revolute">
+    <parent link="link_4" />
+    <child link="link_5" />
+    <origin xyz="0.045 0 0" />
+    <axis xyz="0 0 1" />
+    <limit lower="-2.0944" upper="2.0944" effort="10" velocity="1.0"/>
+</joint>
+<link name="link_6">
+    <visual>
+        <origin xyz="0.01 -0.021 -0.021" rpy="1.57075 0 0"  />
+        <geometry>
+            <mesh filename="file://$(find mecanum_moveit_launch)/meshes/link_6.stl" scale="-0.0003 0.0003 0.0003" />
+        </geometry>
+        <material name="black" />
+    </visual>
+    <collision>
+        <origin xyz="0.02 0 0" rpy="0 1.57075 0"  />
+        <geometry>
+            <cylinder length="0.01" radius="0.016" />
+        </geometry>
+    </collision>
+    <inertial>
+        <mass value="${mass}"/>
+        <inertia ixx="${1/12*mass*(3*radius*radius+length*length)}" ixy="0" ixz="0" iyy="${1/2*mass*radius*radius}" iyz="0" izz="${1/12*mass*(3*radius*radius+length*length)}" />
+    </inertial>
+</link>
+<joint name="rob_joint_6" type="revolute">
+    <parent link="link_5" />
+    <child link="link_6" />
+    <origin xyz="0.033 0 0" rpy="-1.57075 0 0" />
+    <axis xyz="1 0 0" />
+    <limit lower="-6.1087" upper="6.1087" effort="10" velocity="1.0"/>
+</joint>
 <gazebo reference="base_scan">
-<material>Gazebo/Blue</material>
-    <sensor name="lidar_sensor" type="ray">
-        <pose>0 0 0 0 0 0</pose>
-        <visualize>true</visualize>
+<sensor name="base_scan" type="gpu_lidar">
+        <pose relative_to='base_scan'>0 0 0 0 0 0</pose>
+        <topic>scan</topic>
+        <gz_frame_id>base_scan</gz_frame_id>
         <update_rate>10</update_rate>
-        <ray>
-            <scan>
-                <horizontal>
-                    <samples>500</samples>
-                    <resolution>0.72</resolution>
-                    <min_angle>-2.3562</min_angle>
-                    <max_angle>2.3562</max_angle>
-                </horizontal>
-            </scan>
-            <range>
-                <min>0.120</min>
-                <max>10</max>
-                <resolution>0.25</resolution>
-            </range>
-            <noise>
+        <lidar>
+          <scan>
+            <horizontal>
+              <samples>500</samples>
+              <resolution>1</resolution>
+              <min_angle>-2.3562</min_angle>
+              <max_angle>2.3562</max_angle>
+              <!-- <angle_increment>0.0175</angle_increment> -->
+            </horizontal>
+            <!-- <vertical>
+              <samples>1</samples>
+              <resolution>1</resolution>
+              <min_angle>0</min_angle>
+              <max_angle>0</max_angle>
+            </vertical> -->
+          </scan>
+          <range>
+            <min>0.120</min>
+            <max>20.0</max>
+            <resolution>0.25</resolution>
+          </range>
+          <noise>
                 <type>gaussian</type>
                 <mean>0.0</mean>
                 <stddev>0.02</stddev>
-            </noise>
-        </ray>
-        <plugin filename="libgazebo_ros_ray_sensor.so" name="lidar_controller">
-            <frame_name>base_scan</frame_name>
-            <ros>
-                <namespace>/</namespace>
-                <remapping>~/out:=/scan</remapping>
-            </ros>
-            <output_type>sensor_msgs/LaserScan</output_type>
-            <min_intensity>0.0</min_intensity>
-        </plugin>
-    </sensor>
+          </noise>
+          <frame_id>base_scan</frame_id>
+        </lidar>
+        <always_on>1</always_on>
+        <visualize>true</visualize>
+      </sensor>
+    <material>Gazebo/Black</material>
 </gazebo>
+<!-- <gazebo>
+    <plugin filename="libignition-gazebo-sensors-system.so" name="ignition::gazebo::systems::Sensors">
+        <render_engine>ogre</render_engine>
+    </plugin>
+</gazebo> -->
+<gazebo>
+    <plugin
+      filename="libignition-gazebo-mecanum-drive-system.so"
+      name="ignition::gazebo::systems::MecanumDrive">
+      <!-- Topic for the command input -->
+      <topic>/cmd_vel</topic>
+      <!-- Wheel joints -->
+      <front_left_joint>front_left_wheel_joint</front_left_joint>
+      <front_right_joint>front_right_wheel_joint</front_right_joint>
+      <back_left_joint>rear_left_wheel_joint</back_left_joint>
+      <back_right_joint>rear_right_wheel_joint</back_right_joint>
+      <!-- Wheel parameters -->
+      <wheel_separation>0.3</wheel_separation>
+      <wheelbase>0.3</wheelbase>
+      <wheel_radius>0.1</wheel_radius>
+      <!-- Control gains and limits (optional) -->
+      <min_acceleration>-5</min_acceleration>
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