Commit message: joint limitek javítva a description alapján - Marci

File: urdf/mecanum.xacro (robot description, xacro)
@@ -250,5 +250,5 @@
     <origin xyz="0.01 0 0" rpy="-1.57075 0 0"/>
     <axis xyz="0 0 1" />
-    <limit lower="-3.3161" upper="0.7854" effort="10" velocity="1.0"/>
+    <limit lower="-0.7854" upper="0.7854" effort="10" velocity="1.0"/>
 </joint>
 <link name="link_3">
@@ -276,5 +276,5 @@
     <origin xyz="0 -0.090 0" rpy="3.14 0 0" />
     <axis xyz="0 0 1" />
-    <limit lower="-2.0944" upper="2.7227" effort="10" velocity="1.0"/>
+    <limit lower="-1.0472" upper="1.4835" effort="10" velocity="1.0"/>
 </joint>
 <link name="link_4">
@@ -328,5 +328,5 @@
     <origin xyz="0.045 0 0" />
     <axis xyz="0 0 1" />
-    <limit lower="-2.0944" upper="2.0944" effort="10" velocity="1.0"/>
+    <limit lower="-1.5708" upper="1.5708" effort="10" velocity="1.0"/>
 </joint>
 <link name="link_6">

Commit message: dunno

File: urdf/mecanum.xacro (robot description, xacro)
@@ -356,176 +356,3 @@
     <limit lower="-6.1087" upper="6.1087" effort="10" velocity="1.0"/>
 </joint>
-<gazebo reference="base_scan">
-<sensor name="base_scan" type="gpu_lidar">
-        <pose relative_to='base_scan'>0 0 0 0 0 0</pose>
-        <topic>scan</topic>
-        <gz_frame_id>base_scan</gz_frame_id>
-        <update_rate>10</update_rate>
-        <lidar>
-          <scan>
-            <horizontal>
-              <samples>500</samples>
-              <resolution>1</resolution>
-              <min_angle>-2.3562</min_angle>
-              <max_angle>2.3562</max_angle>
-              <!-- <angle_increment>0.0175</angle_increment> -->
-            </horizontal>
-            <!-- <vertical>
-              <samples>1</samples>
-              <resolution>1</resolution>
-              <min_angle>0</min_angle>
-              <max_angle>0</max_angle>
-            </vertical> -->
-          </scan>
-          <range>
-            <min>0.120</min>
-            <max>20.0</max>
-            <resolution>0.25</resolution>
-          </range>
-          <noise>
-                <type>gaussian</type>
-                <mean>0.0</mean>
-                <stddev>0.02</stddev>
-          </noise>
-          <frame_id>base_scan</frame_id>
-        </lidar>
-        <always_on>1</always_on>
-        <visualize>true</visualize>
-      </sensor>
-    <material>Gazebo/Black</material>
-</gazebo>
-<!-- <gazebo>
-    <plugin filename="libignition-gazebo-sensors-system.so" name="ignition::gazebo::systems::Sensors">
-        <render_engine>ogre</render_engine>
-    </plugin>
-</gazebo> -->
-<gazebo>
-    <plugin
-      filename="libignition-gazebo-mecanum-drive-system.so"
-      name="ignition::gazebo::systems::MecanumDrive">
-      <!-- Topic for the command input -->
-      <topic>/cmd_vel</topic>
-      <!-- Wheel joints -->
-      <front_left_joint>front_left_wheel_joint</front_left_joint>
-      <front_right_joint>front_right_wheel_joint</front_right_joint>
-      <back_left_joint>rear_left_wheel_joint</back_left_joint>
-      <back_right_joint>rear_right_wheel_joint</back_right_joint>
-      <!-- Wheel parameters -->
-      <wheel_separation>0.3</wheel_separation>
-      <wheelbase>0.3</wheelbase>
-      <wheel_radius>0.1</wheel_radius>
-      <!-- Control gains and limits (optional) -->
-      <min_acceleration>-5</min_acceleration>
-      <max_acceleration>5</max_acceleration>
-      <!-- Other parameters (optional) -->
-      <odom_topic>odom</odom_topic>
-      <tf_topic>tf</tf_topic>
-      <frame_id>odom</frame_id>
-      <child_frame_id>base_footprint</child_frame_id>
-      <odom_publish_frequency>30</odom_publish_frequency>
-      <publish_odom>true</publish_odom>
-      <publish_odom_tf>true</publish_odom_tf>
-    </plugin>
-    <plugin name="ignition::gazebo::systems::OdometryPublisher" filename="libignition-gazebo-odometry-publisher-system">
-      <odom_topic>odom</odom_topic>
-      <odom_frame>odom</odom_frame>
-      <robot_base_frame>base_footprint</robot_base_frame>
-      <publish_tf>true</publish_tf>
-      <tf_topic>tf</tf_topic>
-      <odom_publish_frequency>30</odom_publish_frequency>
-      <xyz_offset>0 0 0</xyz_offset>
-      <rpy_offset>0 0 0</rpy_offset>
-    </plugin>
-    <plugin
-        filename="libignition-gazebo-joint-state-publisher-system"
-        name="ignition::gazebo::systems::JointStatePublisher">
-        <topic>joint_states</topic>
-        <joint_name>front_left_wheel_joint</joint_name>
-        <joint_name>front_right_wheel_joint</joint_name>
-        <joint_name>rear_left_wheel_joint</joint_name>
-        <joint_name>rear_right_wheel_joint</joint_name>
-    </plugin>
-</gazebo>
-<gazebo reference="front_right_wheel">
-    <collision>
-        <surface>
-            <friction>
-                <ode>
-                    <mu1>1.5</mu1>
-                    <mu2>0</mu2>
-                    <fdir1 ignition:expressed_in="base_footprint">1 1 0</fdir1>
-                </ode>
-            </friction>
-        </surface>
-    </collision>
-    <kp>500000.0</kp>
-    <kd>100.0</kd>
-    <maxVel>0.5</maxVel>
-    <minDepth>0.001</minDepth>
-    <material>Gazebo/Black</material>
-</gazebo>
-<gazebo reference="front_left_wheel">
-    <collision>
-        <surface>
-            <friction>
-                <ode>
-                    <mu1>1.5</mu1>
-                    <mu2>0</mu2>
-                    <fdir1 ignition:expressed_in="base_footprint">1 -1 0</fdir1>
-                </ode>
-            </friction>
-        </surface>
-    </collision>
-    <kp>500000.0</kp>
-    <kd>100.0</kd>
-    <maxVel>0.5</maxVel>
-    <minDepth>0.001</minDepth>
-    <material>Gazebo/Black</material>
-  </gazebo>
-  <gazebo reference="rear_right_wheel">
-    <collision>
-        <surface>
-            <friction>
-                <ode>
-                    <mu1>1.5</mu1>
-                    <mu2>0</mu2>
-                    <fdir1 ignition:expressed_in="base_footprint">1 -1 0</fdir1>
-                </ode>
-            </friction>
-        </surface>
-    </collision>
-    <kp>500000.0</kp>
-    <kd>100.0</kd>
-    <maxVel>0.5</maxVel>
-    <minDepth>0.001</minDepth>
-    <material>Gazebo/Black</material>
-  </gazebo>
-  <gazebo reference="rear_left_wheel">
-    <collision>
-        <surface>
-            <friction>
-                <ode>
-                    <mu1>1.5</mu1>
-                    <mu2>0</mu2>
-                    <fdir1 ignition:expressed_in="base_footprint">1 1 0</fdir1>
-                </ode>
-            </friction>
-        </surface>
-    </collision>
-    <kp>500000.0</kp>
-    <kd>100.0</kd>
-    <maxVel>0.5</maxVel>
-    <minDepth>0.001</minDepth>
-    <material>Gazebo/Black</material>
-  </gazebo>
-  <gazebo reference="base_link">
-    <material>Gazebo/Yellow</material>
-    <mu1>0.000002</mu1>
-    <mu2>0.000002</mu2>
-  </gazebo>
-  <gazebo reference="link_0">
-    <material>Gazebo/Orange</material>
-    <mu1>0.000002</mu1>
-    <mu2>0.000002</mu2>
-  </gazebo>
 </robot>

Commit message: MoveIt2 + valós robot mozgatás, forgatáshoz használt verzió, javított joint_states_publisherrel, fix kerék jointokkal

File: urdf/mecanum.xacro (robot description, xacro)
@@ -43,5 +43,5 @@
     </inertial>
 </link>
-<joint name="front_right_wheel_joint" type="continuous">
+<joint name="front_right_wheel_joint" type="fixed">
     <parent link="base_link" />
     <child link="front_right_wheel" />
@@ -68,5 +68,5 @@
     </inertial>
 </link>
-<joint name="front_left_wheel_joint" type="continuous">
+<joint name="front_left_wheel_joint" type="fixed">
     <parent link="base_link" />
     <child link="front_left_wheel" />
@@ -93,5 +93,5 @@
     </inertial>
 </link>
-<joint name="rear_left_wheel_joint" type="continuous">
+<joint name="rear_left_wheel_joint" type="fixed">
     <parent link="base_link" />
     <child link="rear_left_wheel" />
@@ -118,5 +118,5 @@
     </inertial>
 </link>
-<joint name="rear_right_wheel_joint" type="continuous">
+<joint name="rear_right_wheel_joint" type="fixed">
     <parent link="base_link" />
     <child link="rear_right_wheel" />

Commit message: Lidar orange

File: urdf/mecanum.xacro (robot description, xacro)
@@ -156,5 +156,5 @@
             <mesh filename="file://$(find mecanum_moveit_launch)/meshes/sensors/hokuyo_ust10.stl" scale="0.8 0.8 0.8" />
         </geometry>
-        <material name="black" />
+        <material name="orange" />
     </visual>
     <collision>

Commit message: Final commit (mesh file correction)

File: urdf/mecanum.xacro (robot description, xacro)
@@ -179,5 +179,5 @@
         <origin xyz="-0.005 0.010 -0.035" rpy="1.57075 0 0"  />
         <geometry>
-            <mesh filename="file://$(find mecanum_moveit_launch)/meshes/simplify_link_0.stl" scale="0.0003 0.0003 0.0003" />
+            <mesh filename="file://$(find mecanum_moveit_launch)/meshes/link_0.stl" scale="0.0003 0.0003 0.0003" />
         </geometry>
         <material name="black" />
@@ -204,5 +204,5 @@
         <origin xyz="-0.020 -0.030 -0.065" rpy="1.57075 0 0"  />
         <geometry>
-            <mesh filename="file://$(find mecanum_moveit_launch)/meshes/simplify_link_1.stl" scale="-0.0003 0.0003 0.0003" />
+            <mesh filename="file://$(find mecanum_moveit_launch)/meshes/link_1.stl" scale="-0.0003 0.0003 0.0003" />
         </geometry>
         <material name="orange" />
@@ -230,5 +230,5 @@
         <origin xyz="0.005 -0.115 0.048" rpy="0 0 0"  />
         <geometry>
-            <mesh filename="file://$(find mecanum_moveit_launch)/meshes/simplify_link_2.stl" scale="-0.0003 0.0003 0.0003" />
+            <mesh filename="file://$(find mecanum_moveit_launch)/meshes/link_2.stl" scale="-0.0003 0.0003 0.0003" />
         </geometry>
         <material name="orange" />
@@ -256,5 +256,5 @@
         <origin xyz="0.015 -0.025 0.0235" rpy="0 0 0"  />
         <geometry>
-            <mesh filename="file://$(find mecanum_moveit_launch)/meshes/simplify_link_3.stl" scale="-0.0003 0.0003 0.0003" />
+            <mesh filename="file://$(find mecanum_moveit_launch)/meshes/link_3.stl" scale="-0.0003 0.0003 0.0003" />
         </geometry>
         <material name="orange" />
@@ -282,5 +282,5 @@
         <origin xyz="0.04 -0.020 0.015" rpy="0 0 0"  />
         <geometry>
-            <mesh filename="file://$(find mecanum_moveit_launch)/meshes/simplify_link_4.stl" scale="-0.0003 0.0003 0.0003" />
+            <mesh filename="file://$(find mecanum_moveit_launch)/meshes/link_4.stl" scale="-0.0003 0.0003 0.0003" />
         </geometry>
         <material name="orange" />
@@ -308,5 +308,5 @@
         <origin xyz="0.020 -0.02 0.02" rpy="0 0 0"  />
         <geometry>
-            <mesh filename="file://$(find mecanum_moveit_launch)/meshes/simplify_link_5.stl" scale="-0.0003 0.0003 0.0003" />
+            <mesh filename="file://$(find mecanum_moveit_launch)/meshes/link_5.stl" scale="-0.0003 0.0003 0.0003" />
         </geometry>
         <material name="orange" />

Commit message: Final commit (mecanum.stl)

File: urdf/mecanum.xacro (robot description, xacro)
@@ -28,5 +28,5 @@
         <origin xyz="0 0 0" rpy="1.57075 0 0"  />
         <geometry>
-            <mesh filename="file://$(find mecanum_moveit_launch)/meshes/Mecanum_jo.stl" scale="0.0010 0.0010 0.0010" />
+            <mesh filename="file://$(find mecanum_moveit_launch)/meshes/Mecanum.stl" scale="0.0010 0.0010 0.0010" />
         </geometry>
         <material name="black" />
@@ -53,5 +53,5 @@
         <origin xyz="0 0 0" rpy="1.57075 0 0"  />
         <geometry>
-            <mesh filename="file://$(find mecanum_moveit_launch)/meshes/Mecanum_jo.stl" scale="0.0010 0.0010 0.0010" />
+            <mesh filename="file://$(find mecanum_moveit_launch)/meshes/Mecanum.stl" scale="0.0010 0.0010 0.0010" />
         </geometry>
         <material name="black" />
@@ -78,5 +78,5 @@
         <origin xyz="0 0 0" rpy="1.57075 0 0"  />
         <geometry>
-            <mesh filename="file://$(find mecanum_moveit_launch)/meshes/Mecanum_jo.stl" scale="0.0010 0.0010 0.0010" />
+            <mesh filename="file://$(find mecanum_moveit_launch)/meshes/Mecanum.stl" scale="0.0010 0.0010 0.0010" />
         </geometry>
         <material name="black" />
@@ -103,5 +103,5 @@
         <origin xyz="0 0 0" rpy="1.57075 0 0"  />
         <geometry>
-            <mesh filename="file://$(find mecanum_moveit_launch)/meshes/Mecanum_jo.stl" scale="0.0010 0.0010 0.0010" />
+            <mesh filename="file://$(find mecanum_moveit_launch)/meshes/Mecanum.stl" scale="0.0010 0.0010 0.0010" />
         </geometry>
         <material name="black" />
